File: rgb_led_attiny.sch (EAGLE design)
At the start: 5 parts, among them IC1 ATTINY45-20PU, IC2 MC7805BTG

Commit message: Premier jet du schematic
Parts:
- added JP2, JP3, JP4: (no value), pinhead:PINHD-1X2
- added Q1, Q2, Q3: IRF540NPBF, rgb_led_attiny:IRF540NPBF
- added R1, R2, R3: (no value), rcl:R-EU_0613/15
Connections:
- new net N$2: Q2.D, R2.1
- new net N$3: Q1.D, R1.1
- new net N$4: JP2.1, R1.2
- new net N$5: JP3.1, R2.2
- new net N$6: Q3.D, R3.1
- new net N$7: JP4.1, R3.2
- new net PWM_B: IC1.PB0, Q3.G
- new net PWM_G: IC1.PB1, Q2.G
- new net PWM_R: IC1.PB2, Q1.G
- net GND: now also IC1.GND, Q1.S, Q2.S, Q3.S
- net VCC: now also IC1.VCC, JP2.2, JP3.2, JP4.2
Other:
- moved on the sheet: C1, C2, IC1, IC2, JP1
